Commit message: Adjusted max angles on the robot's arm.

File: test_robots/urdf/bot.urdf (robot description, URDF)
Before this commit: robot aerial_manipulator_drone, 5 links, 4 joints
Joints:
- joint arm2_hinge: limit lower=-0.5 upper=0.5 effort=1000.0 velocity=0.5 -> lower=-1.0 upper=1.0 effort=1000.0 velocity=0.5
- joint arm3_hinge: limit lower=-0.5 upper=0.5 effort=1000.0 velocity=0.5 -> lower=-1.0 upper=1.0 effort=1000.0 velocity=0.5
- joint arm_hinge: limit lower=-0.5 upper=0.5 effort=1000.0 velocity=0.5 -> lower=-1.0 upper=1.0 effort=1000.0 velocity=0.5

Commit message: Made the drone a bit more realistically-sized.

File: test_robots/urdf/bot.urdf (robot description, URDF)
Before this commit: robot aerial_manipulator_drone, 5 links, 4 joints
Links:
- link arm: geometry collision box size=0.01 0.25 0.01; visual box size=0.01 0.25 0.01
- link arm2: geometry collision box size=0.01 0.25 0.01; visual box size=0.01 0.25 0.01
- link arm3: geometry collision box size=0.01 0.25 0.01; visual box size=0.01 0.25 0.01
- link end_effector: geometry visual box size=0.08 0.08 0.08
Joints:
- joint arm2_hinge: origin xyz=0.0 0.5 0.0 -> xyz=0.0 0.25 0.0
- joint arm3_hinge: origin xyz=0.0 0.5 0.0 -> xyz=0.0 0.25 0.0
- joint arm_hinge: origin xyz=0.0 0.1750 0.0 -> xyz=0.0 0.2 0.0
- joint end_effector_joint: origin xyz=0.0 0.5 0.0 -> xyz=0.0 0.25 0.0

Commit message: Made the bot arm slightly thicker

File: test_robots/urdf/bot.urdf (robot description, URDF)
Before this commit: robot aerial_manipulator_drone, 5 links, 4 joints
Links:
- link arm: geometry collision box size=0.05 0.25 0.05; visual box size=0.05 0.25 0.05
- link arm2: geometry collision box size=0.05 0.25 0.05; visual box size=0.05 0.25 0.05
- link arm3: geometry collision box size=0.05 0.25 0.05; visual box size=0.05 0.25 0.05

Commit message: Drone model!

File: test_robots/urdf/bot.urdf (robot description, URDF)
Before this commit: robot aerial_manipulator_drone, 5 links, 4 joints
Links:
- link base_link: geometry collision box size=0.4 0.4 0.2; visual mesh filename=test_robots/meshes/drone.dae

Commit message: Refactored, beautified, and made a video.

File: test_robots/urdf/bot.urdf (robot description, URDF)
Before this commit: robot aerial_manipulator_drone, 5 links, 4 joints
Links:
- link base_link: geometry collision box size=0.8 0.8 0.2; visual mesh filename=test_robots/meshes/drone.dae

Commit message: Poked a bit at the goal sample construction bits.
Signed-off-by: Werner Kroneman <w.kroneman@ucr.nl>

File: test_robots/urdf/bot.urdf (robot description, URDF)
Before this commit: robot aerial_manipulator_drone, 5 links, 4 joints
Joints:
- joint end_effector_joint: axis 0 1 0 -> (none); type continuous -> fixed
